File: SARA-R4_DevBoard.kicad_pcb (KiCad board)
At the start: 4 copper layers, 60 x 38 mm, 54 parts, among them J1 JAE_SIM_Card_SF72S006, J2 Battery connector, J3 USB4110-GF-A, J4 SWD connector, U1 SARA-R422X, U2 STM32L432KCUx, U3 ESD224DQAR, U4 MCP73831, U5 SiP32431DR3, U6 TPS7A0218PDBVR, Y1 32.768kHz

Commit message: Force update
Parts:
- removed the REF** at (168.6, 85.0)
- removed S1: PTS526_SM15_SMTR2_LFS, SARA-R4_DevBoard-lib:PTS526SM15SMTR2LFS
- added C22: 6.8pF, Capacitor_SMD:C_0402_1005Metric, B.Cu at (162.5, 105.0)
- added C25: 68pF, Capacitor_SMD:C_0402_1005Metric, F.Cu at (146.0, 94.2)
- added C26: 10nF, Capacitor_SMD:C_0402_1005Metric, F.Cu at (146.0, 93.2)
- added C27: 0.1uF, Capacitor_SMD:C_0402_1005Metric, F.Cu at (143.6, 92.3)
- added C28: 10uF, Capacitor_SMD:C_0402_1005Metric, F.Cu at (146.0, 92.2)
- added C29: 2.2pF, Capacitor_SMD:C_0402_1005Metric, F.Cu at (135.9, 102.5)
- added C30: 0.5pF, Capacitor_SMD:C_0402_1005Metric, F.Cu at (141.0, 103.0)
- added C31: DNP, Capacitor_SMD:C_0402_1005Metric, F.Cu at (137.7, 103.0)
- added C32: 0.1uF, Capacitor_SMD:C_0402_1005Metric, F.Cu at (165.1, 91.5)
- added FB2: FerriteBead_Small, Inductor_SMD:L_0603_1608Metric, F.Cu at (144.3, 95.9)
- added J5: I2C Ext. Conn., Connector_JST:JST_SH_SM04B-SRSS-TB_1x04-1MP_P1.00mm_Horizontal, B.Cu at (174.7, 83.6)
- added L5: 15nH, Inductor_SMD:L_0402_1005Metric, F.Cu at (134.3, 103.0)
- added L6: 15nH, Inductor_SMD:L_0402_1005Metric, F.Cu at (133.7, 97.5)
- added R10: 4.7k, Resistor_SMD:R_0402_1005Metric, B.Cu at (155.3, 98.2)
- added R11: 10k, Resistor_SMD:R_0402_1005Metric, B.Cu at (150.1, 116.9)
- added R12: 60, Resistor_SMD:R_0402_1005Metric, B.Cu at (164.6, 114.8)
- added R13: 60, Resistor_SMD:R_0402_1005Metric, B.Cu at (162.4, 114.8)
- added R7: 5.1k, Resistor_SMD:R_0402_1005Metric, B.Cu at (155.9, 81.7)
- added R8: 10k, Resistor_SMD:R_0402_1005Metric, B.Cu at (158.7, 106.7)
- added R9: 4.7k, Resistor_SMD:R_0402_1005Metric, B.Cu at (154.8, 99.3)
- added TP10: TestPoint, TestPoint:TestPoint_Pad_D1.0mm, F.Cu at (146.9, 115.5)
- added TP11: TestPoint, TestPoint:TestPoint_Pad_D1.0mm, F.Cu at (162.4, 116.6)
- added TP12: USB_D+, TestPoint:TestPoint_Pad_D1.0mm, F.Cu at (175.0, 117.0)
- added TP13: TestPoint, TestPoint:TestPoint_Pad_D1.0mm, F.Cu at (153.6, 94.7)
- added TP14: TestPoint, TestPoint:TestPoint_Pad_D1.0mm, F.Cu at (154.5, 118.0)
- added TP15: USB_D-, TestPoint:TestPoint_Pad_D1.0mm, F.Cu at (172.0, 117.0)
- added TP16: TestPoint, TestPoint:TestPoint_Pad_D1.0mm, F.Cu at (150.7, 96.4)
- added TP17: TestPoint, TestPoint:TestPoint_Pad_D1.0mm, F.Cu at (153.9, 115.1)
- added TP18: SARA_USB_5V0, TestPoint:TestPoint_Pad_D1.0mm, F.Cu at (169.0, 117.0)
- added TP19: TestPoint, TestPoint:TestPoint_Pad_D1.0mm, F.Cu at (170.4, 91.2)
- added TP20: TestPoint, TestPoint:TestPoint_Pad_D1.0mm, F.Cu at (157.3, 115.1)
- added TP21: SARA_USB_5V0, TestPoint:TestPoint_Pad_D1.0mm, F.Cu at (178.0, 117.0)
- added TP22: TestPoint, TestPoint:TestPoint_Pad_D1.0mm, F.Cu at (170.5, 93.3)
- added TP23: TestPoint, TestPoint:TestPoint_Pad_D1.0mm, F.Cu at (157.5, 118.0)
- added TP3: 1V8, TestPoint:TestPoint_Pad_D1.0mm, B.Cu at (142.3, 105.5)
- added TP4: 5V, TestPoint:TestPoint_Pad_D1.0mm, B.Cu at (174.1, 95.2)
- added TP5: 5V, TestPoint:TestPoint_Pad_D1.0mm, F.Cu at (138.0, 94.6)
- added TP6: 5V, TestPoint:TestPoint_Pad_D1.0mm, F.Cu at (138.0, 91.7)
- added TP7: VBUS, TestPoint:TestPoint_Pad_D1.0mm, B.Cu at (149.7, 90.6)
- added TP8: UART1_TX, TestPoint:TestPoint_Pad_D1.0mm, B.Cu at (139.4, 91.5)
- added TP9: UART1_RX, TestPoint:TestPoint_Pad_D1.0mm, B.Cu at (139.4, 87.5)
- added U10: SARA-R422X, RF_GSM:ublox_SARA-G3_LGA-96, F.Cu at (155.1, 105.8)
- added U11: SIM-ST-MFF2, Package_DFN_QFN:DFN-8-1EP_6x5mm_P1.27mm_EP4x4mm, F.Cu at (160.0, 93.9)
- added U7: MX25R6435FZNIL0, Package_SON:WSON-8-1EP_4x4mm_P0.8mm_EP2.2x3mm, B.Cu at (150.1, 113.8)
- added U8: TCAN1044VDDFRQ1, SARA-R4_DevBoard_Library:SOT65P280X110-8N, B.Cu at (163.5, 110.7)
- added U9: LIS2DH, Package_LGA:LGA-14_2x2mm_P0.35mm_LayoutBorder3x4y, B.Cu at (160.0, 93.9)
- ANT1: footprint SARA-R4_DevBoard-lib:SR4L002 -> SARA-R4_DevBoard_Library:SR4L002
- ANT2: footprint SARA-R4_DevBoard-lib:SR4G008 -> SARA-R4_DevBoard_Library:SR4G008
- C1: value 100nF -> 1.5pF; footprint Capacitor_SMD:C_0603_1608Metric -> Capacitor_SMD:C_0402_1005Metric; moved to F.Cu
- C10: value 47nF -> 0.1uF
- C11: value 15pF -> 0.1uF
- C12, C13, C15: value 47nF -> 0.1uF; moved to B.Cu
- C14: value 68pF -> 0.1uF; moved to B.Cu
- C16: value 10nF -> 0.1uF; moved to B.Cu
- C17, C9: value 100nF -> 0.1uF; footprint Capacitor_SMD:C_0603_1608Metric -> Capacitor_SMD:C_0402_1005Metric; moved to B.Cu
- C18: value 10uF -> 0.1uF; moved to B.Cu
- C19: value 100nF -> 0.1uF; footprint Capacitor_SMD:C_0603_1608Metric -> Capacitor_SMD:C_0402_1005Metric
- C2, C3: value 6.8pF -> 4.7uF; footprint Capacitor_SMD:C_0603_1608Metric -> Capacitor_SMD:C_0402_1005Metric; moved to F.Cu
- C20: value 100nF -> 4.7uF; footprint Capacitor_SMD:C_0603_1608Metric -> Capacitor_SMD:C_0402_1005Metric
- C21: value 100nF -> 6.8pF; footprint Capacitor_SMD:C_0603_1608Metric -> Capacitor_SMD:C_0402_1005Metric
- C23: value 1uF -> 0.1uF; footprint Capacitor_SMD:C_0603_1608Metric -> Capacitor_SMD:C_0402_1005Metric
- C24: value 1uF -> 15pF; footprint Capacitor_SMD:C_0603_1608Metric -> Capacitor_SMD:C_0402_1005Metric; moved to F.Cu
- C4: value C_Small -> 10uF; moved to B.Cu
- C5: value C_Small -> 22uF; moved to B.Cu
- C6: value DNP -> 0.1uF; moved to B.Cu
- C7, C8: value C_Small -> 1uF; moved to B.Cu
- D1: value RED LED -> BAT60A; footprint LED_SMD:LED_0402_1005Metric -> Diode_SMD:D_SOD-323; moved to F.Cu
- D2: value GREEN LED -> SZNUP2115LT1G; footprint LED_SMD:LED_0402_1005Metric -> Package_TO_SOT_SMD:SOT-23; moved to B.Cu
- FB1: value FerriteBead_Small -> USB_Bead
- J1: value JAE_SIM_Card_SF72S006 -> Battery; footprint Connector_JAE:JAE_SIM_Card_SF72S006 -> Connector_JST:JST_PH_S2B-PH-SM4-TB_1x02-1MP_P2.00mm_Horizontal
- J2: value Battery connector -> USB4110-GF-A; footprint Connector_JST:JST_SH_BM02B-SRSS-TB_1x02-1MP_P1.00mm_Vertical -> SARA-R4_DevBoard_Library:GCT_USB4110-GF-A_REVB
- J3: value USB4110-GF-A -> SPI Ext. Conn.; footprint SARA-R4_DevBoard-lib:GCT_USB4110-GF-A_REVB -> Connector_JST:JST_SH_SM06B-SRSS-TB_1x06-1MP_P1.00mm_Horizontal; moved to B.Cu
- J4: value SWD connector -> SWD/IO Ext. Conn.; footprint Connector:Tag-Connect_TC2030-IDC-NL_2x03_P1.27mm_Vertical -> Connector_JST:JST_SH_SM04B-SRSS-TB_1x04-1MP_P1.00mm_Horizontal
- L1: value 3.3nH -> L_Small
- L2: value L_Small -> 12nH
- L3: value 15nH -> 4.7uH; moved to B.Cu
- L4: value 15nH -> 3.3nH
- R1: value 10k -> 1.13k; moved to F.Cu
- R2: value 5.1k -> 1.18k; moved to F.Cu
- R3: value 5.1k -> 1.13k; moved to F.Cu
- R4: value 2k -> 18k; moved to F.Cu
- R5: value 470 -> 5.1k
- R6: value 470 -> 5.1k; moved to B.Cu
- REF**: moved to F.Cu
- U1: value SARA-R422X -> BQ24075RGT; footprint RF_GSM:ublox_SARA-G3_LGA-96 -> Package_DFN_QFN:VQFN-16-1EP_3x3mm_P0.5mm_EP1.6x1.6mm
- U2: value STM32L432KCUx -> TPS7A0218; footprint Package_DFN_QFN:QFN-32-1EP_5x5mm_P0.5mm_EP3.45x3.45mm -> Package_TO_SOT_SMD:SOT-23-5
- U3: value ESD224DQAR -> TPS613222ADBV; footprint SARA-R4_DevBoard-lib:ESD224DQAR -> Package_TO_SOT_SMD:SOT-23-5; moved to B.Cu
- U4: value MCP73831 -> FT230XQ; footprint Package_TO_SOT_SMD:SOT-23-5 -> Package_DFN_QFN:QFN-16-1EP_4x4mm_P0.65mm_EP2.1x2.1mm; moved to B.Cu
- U5: value SiP32431DR3 -> USBLC6; footprint Package_TO_SOT_SMD:SOT-363_SC-70-6 -> Package_TO_SOT_SMD:SOT-23-6; moved to B.Cu
- U6: value TPS7A0218PDBVR -> STM32L432KCUx; footprint Package_TO_SOT_SMD:SOT-23-5 -> Package_DFN_QFN:QFN-32-1EP_5x5mm_P0.5mm_EP3.45x3.45mm
- Y1: footprint SARA-R4_DevBoard-lib:NX3215SA32768KEXS00AMU00003 -> SARA-R4_DevBoard_Library:NX3215SA32768KEXS00AMU00003
- moved D2 45.5 mm to (163.5, 117.6), turned to -90 degrees
- moved L3 33.4 mm to (166.8, 97.1), turned to 180 degrees
- moved L1 29.9 mm to (169.0, 101.9), turned to 90 degrees
- moved C6 28.5 mm to (165.4, 97.6)
- moved J1 27.6 mm to (140.6, 85.8), turned to 90 degrees
- moved C3 27.2 mm to (141.2, 84.5)
- moved J4 26.1 mm to (142.3, 116.5), turned to 180 degrees
- moved C4 25.3 mm to (165.4, 95.5)
- moved C23 25.1 mm to (165.7, 110.2), turned to 90 degrees
- moved C16 24.4 mm to (166.6, 87.5), turned to 0 degrees
- moved C8 24.2 mm to (149.8, 108.2)
- moved C12 23.2 mm to (147.8, 108.2), turned to -90 degrees
- moved C14 22.5 mm to (158.2, 108.1), turned to -90 degrees
- moved J3 22.2 mm to (164.6, 83.6), turned to 0 degrees
- moved C17 21.3 mm to (160.2, 107.2), turned to -90 degrees
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Connections:
- ANT1 pad 4: Net-(ANT1-Pad4) -> Net-(ANT1-RETURN/GND)
- C1 pad 1: /NRST -> Net-(U10-ANT_GNSS)
- C1 pad 2: GND -> /RF_GNSS_FEED
- C10 pad 1: GND -> /VBUS
- C10 pad 2: /VSIM -> GND
- C11 pad 1: /SARA_VCC -> Net-(C11-Pad1)
- C12 pad 1: GND -> +1V8
- C12 pad 2: /SIM_RST -> GND
- C13 pad 1: GND -> +1V8
- C13 pad 2: /SIM_IO -> GND
- C14 pad 1: /SARA_VCC -> +1V8
- C15 pad 1: GND -> +5V
- C15 pad 2: /SIM_CLK -> GND
- C16 pad 1: /SARA_VCC -> +5V
- C17 pad 1: /SARA_VCC -> /NRST
- C18 pad 1: /SARA_VCC -> GND
- C18 pad 2: GND -> +1V8
- C2 pad 1: /OSC_32_IN -> VSYS
- C20 pad 1: +1V8 -> GND
- C20 pad 2: GND -> Net-(C20-Pad2)
- C21 pad 1: +1V8 -> /OSC_32_IN
- C23 pad 1: +1V8 -> +5V
- C24 pad 1: +BATT -> VSYS
- C3 pad 1: /OSC_32_OUT -> +BATT
- C4 pad 1: /RF_GSM -> GND
- C4 pad 2: GND -> VSYS
- C5 pad 1: /RF_GNSS -> +5V
- C6 pad 1: Net-(C6-Pad1) -> VSYS
- C7 pad 1: Net-(C6-Pad1) -> VSYS
- C7 pad 2: /RF_GSM_FEED -> GND
- C8 pad 1: /RF_GNSS_FEED -> +1V8
- C9 pad 1: GND -> +1V8
- C9 pad 2: /VSIM -> GND
- D1 pad 1: Net-(D1-Pad1) -> VDC
- D1 pad 2: VBUS -> /VBUS
- D2 pad 1: Net-(D2-Pad1) -> /CAN_L
- D2 pad 2: GND -> /CAN_H
- FB1 pad 1: /SARA_VCC -> /VBUS
- FB1 pad 2: VCC -> Net-(C11-Pad1)
- J4 pad 1: +1V8 -> unconnected-(J4-Pin_1-Pad1)
- J4 pad 2: /SWDIO -> /SWDIO/IO2
- J4 pad 3: /NRST -> /SWCLK/IO3
- J4 pad 4: /(LPTIM1_OUT) -> GND
- L1 pad 1: /RF_GSM -> GND
- L1 pad 2: Net-(C6-Pad1) -> Net-(U10-ANT_GNSS)
- L2 pad 1: /RF_GNSS -> GND
- L3 pad 1: GND -> Net-(U3-SW)
- L3 pad 2: /RF_GSM_FEED -> VSYS
- L4 pad 1: GND -> /RF_GSM
- L4 pad 2: Net-(ANT1-Pad4) -> Net-(C29-Pad1)
- R1 pad 1: Net-(R1-Pad1) -> Net-(U1-TMR)
- R1 pad 2: /BOOT -> GND
- R2 pad 1: GND -> Net-(U1-ILIM)
- R2 pad 2: Net-(J3-PadA5) -> GND
- R3 pad 1: GND -> Net-(U1-ISET)
- R3 pad 2: Net-(J3-PadB5) -> GND
- R4 pad 1: Net-(R4-Pad1) -> Net-(U1-TS)
- R5 pad 1: Net-(D1-Pad1) -> /VBUS
- R5 pad 2: Net-(R5-Pad2) -> GND
- R6 pad 1: Net-(R5-Pad2) -> GND
- R6 pad 2: Net-(D2-Pad1) -> Net-(J2-CC1)
- U1 pad 1: GND -> Net-(U1-TS)
- U1 pad 10: unconnected-(U1-Pad10) -> VSYS
- U1 pad 11: unconnected-(U1-Pad11) -> VSYS
- U1 pad 12: /UART1_RX -> Net-(U1-ILIM)
- U1 pad 13: /UART1_TX -> VDC
- U1 pad 14: GND -> Net-(U1-TMR)
- U1 pad 15: /PWR_CTRL -> GND
- U1 pad 16: unconnected-(U1-Pad16) -> Net-(U1-ISET)
- U1 pad 17: unconnected-(U1-Pad17) -> GND
- U1 pad 2: unconnected-(U1-Pad2) -> +BATT
- U1 pad 3: GND -> +BATT
- U1 pad 4: /V_INT -> /BOOT/CE
- U1 pad 5: GND -> VSYS
- U1 pad 6: unconnected-(U1-Pad6) -> GND
- U1 pad 7: unconnected-(U1-Pad7) -> /PGOOD
- U1 pad 8: unconnected-(U1-Pad8) -> GND
- U1 pad 9: unconnected-(U1-Pad9) -> /CHG
- U2 pad 1: +1V8 -> VSYS
- U2 pad 2: /OSC_32_IN -> GND
- U2 pad 3: /OSC_32_OUT -> VSYS
- U2 pad 4: /NRST -> unconnected-(U2-NC-Pad4)
- U3 pad 1: /VSIM -> Net-(U3-SW)
- U3 pad 2: /SIM_RST -> GND
- U3 pad 3: GND -> unconnected-(U3-NC-Pad3)
- U3 pad 4: /SIM_IO -> +5V
- U3 pad 5: /SIM_CLK -> unconnected-(U3-NC-Pad5)
- U4 pad 1: Net-(R5-Pad2) -> +1V8
- U4 pad 2: GND -> /UART1_RX
- U4 pad 3: +BATT -> GND
- U4 pad 4: VBUS -> unconnected-(U4-~{CTS}-Pad4)
- U4 pad 5: Net-(R4-Pad1) -> unconnected-(U4-CBUS2-Pad5)
- U5 pad 1: /SARA_VCC -> Net-(U4-USBDP)
- U5 pad 3: /VBAT_CTRL -> /USB_D+
- U5 pad 4: +BATT -> /USB_D-
- U5 pad 5: GND -> /VBUS
- U5 pad 6: unconnected-(U5-Pad6) -> Net-(U4-USBDM)
- U6 pad 1: +BATT -> +1V8
- U6 pad 2: GND -> /OSC_32_IN
- U6 pad 3: +BATT -> /OSC_32_OUT
- U6 pad 4: GND -> /NRST
Routing:
- net VSYS: track 0.00 -> 55.7 mm, vias 0 -> 8
- net +5V: track 0.00 -> 52.6 mm
- net /I2C1_SDA: track 0.00 -> 36.9 mm
- net /I2C1_SCL: track 0.00 -> 36.3 mm, vias 0 -> 2
- net /UART1_RX: track 0.00 -> 28.1 mm, vias 1 -> 2
- net /UART1_TX: track 0.00 -> 27.8 mm, vias 1 -> 0
- net /SPI3_NSS: track 0.00 -> 27.3 mm
- net /BOOT/CE: track 0.00 -> 26.1 mm, vias 0 -> 3
- net /SPI3_MISO: track 0.00 -> 25.9 mm
- net /IMU_INT1: track 0.00 -> 23.0 mm, vias 0 -> 2
- net /SPI3_MOSI: track 0.00 -> 22.2 mm
- net /SPI3_SCK: track 0.00 -> 21.6 mm
- net /UART2_CTS: track 0.00 -> 21.3 mm, vias 0 -> 1
- net /CAN_RX: track 0.00 -> 19.8 mm, vias 0 -> 2
- net Net-(J1-PadC3): track 19.5 -> 0.00 mm
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- added copper zone on B.Cu, net /VBUS
- added copper zone on F.Cu, net /VBUS
- added copper zone on F.Cu, net VDC
- added copper zone on B.Cu, net VSYS
- added copper zone on F.Cu, net VSYS
- added copper zone on In2.Cu, net VSYS
- removed copper zone on B.Cu, net +BATT
- removed copper zone on F.Cu, net /RF_GSM_FEED
- removed copper zone on F.Cu, net /SARA_VCC
- removed copper zone on B.Cu, net VBUS
- removed copper zone on F.Cu, net VBUS
Other:
- board size 60 x 38 mm -> 60 x 40 mm
- board text added: "X"
- board text added: "Y"
- board text added: "Z"
- board text removed: "SARA-R4 IOT dev board"

Commit message: Remove backups and update gerbers
Parts:
- added REF**: TestPoint_Pad_2.0x2.0mm, TestPoint:TestPoint_Pad_2.0x2.0mm, B.Cu at (166.1, 118.4)
- added REF**: TestPoint_Pad_2.0x2.0mm, TestPoint:TestPoint_Pad_2.0x2.0mm, B.Cu at (160.9, 118.4)
Routing:
- net /CAN_L: track 6.96 -> 9.42 mm
- net /CAN_H: track 6.97 -> 9.41 mm
- net GND: vias 195 -> 194
Changed lines of the file:
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@@
       (usegerberextensions true)
       (usegerberattributes true)
-      (usegerberadvancedattributes true)
-      (creategerberjobfile true)
+      (usegerberadvancedattributes false)
+      (creategerberjobfile false)
       (dashed_line_dash_ratio 12.000000)
       (dashed_line_gap_ratio 3.000000)
@@
       (psa4output false)
       (plotreference true)
-      (plotvalue true)
+      (plotvalue false)
       (plotinvisibletext false)
       (sketchpadsonfab false)
@@
     )
   )
+  (footprint "TestPoint:TestPoint_Pad_2.0x2.0mm" (layer "B.Cu")
+    (at 166.1 118.4 180)
+    (descr "SMD rectangular pad as test Point, square 2.0mm side length")
+    (tags "test point SMD pad rectangle square")
+    (attr exclude_from_pos_files exclude_from_bom)
+    (fp_text reference "REF**" (at 0 1.998) (layer "B.SilkS")
+        (effects (font (size 1 1) (thickness 0.15)) (justify mirror))
+    )
+    (fp_text value "TestPoint_Pad_2.0x2.0mm" (at 0 -2.05) (layer "B.Fab")
+        (effects (font (size 1 1) (thickness 0.15)) (justify mirror))
+    )
+    (fp_text user "${REFERENCE}" (at 0 2) (layer "B.Fab")
+        (effects (font (size 1 1) (thickness 0.15)) (justify mirror))
+    )
+    (fp_line (start -1.2 -1.2) (end -1.2 1.2)
+      (stroke (width 0.12) (type solid)) (layer "B.SilkS"))
+    (fp_line (start -1.2 1.2) (end 1.2 1.2)
+      (stroke (width 0.12) (type solid)) (layer "B.SilkS"))
+    (fp_line (start 1.2 -1.2) (end -1.2 -1.2)
+      (stroke (width 0.12) (type solid)) (layer "B.SilkS"))
+    (fp_line (start 1.2 1.2) (end 1.2 -1.2)
+      (stroke (width 0.12) (type solid)) (layer "B.SilkS"))
+    (fp_line (start -1.5 1.5) (end -1.5 -1.5)
+      (stroke (width 0.05) (type solid)) (layer "B.CrtYd"))
+    (fp_line (start -1.5 1.5) (end 1.5 1.5)
+      (stroke (width 0.05) (type solid)) (layer "B.CrtYd"))
+    (fp_line (start 1.5 -1.5) (end -1.5 -1.5)
+      (stroke (width 0.05) (type solid)) (layer "B.CrtYd"))
+    (fp_line (start 1.5 -1.5) (end 1.5 1.5)
+      (stroke (width 0.05) (type solid)) (layer "B.CrtYd"))
+    (pad "1" smd rect (at 0 0 180) (size 2 2) (layers "B.Cu" "B.Mask")
+      (net 11 "/CAN_H"))
+  )
   (footprint "Connector_JST:JST_SH_SM04B-SRSS-TB_1x04-1MP_P1.00mm_Horizontal" (layer "B.Cu")
     (at 174.73 83.6)
@@
     )
   )
+  (footprint "TestPoint:TestPoint_Pad_2.0x2.0mm" (layer "B.Cu")
+    (at 160.9 118.4 180)
+    (descr "SMD rectangular pad as test Point, square 2.0mm side length")
+    (tags "test point SMD pad rectangle square")
+    (attr exclude_from_pos_files exclude_from_bom)
+    (fp_text reference "REF**" (at 0 1.998) (layer "B.SilkS")
+        (effects (font (size 1 1) (thickness 0.15)) (justify mirror))
+    )
+    (fp_text value "TestPoint_Pad_2.0x2.0mm" (at 0 -2.05) (layer "B.Fab")
+        (effects (font (size 1 1) (thickness 0.15)) (justify mirror))
+    )
+    (fp_text user "${REFERENCE}" (at 0 2) (layer "B.Fab")
+        (effects (font (size 1 1) (thickness 0.15)) (justify mirror))
+    )
+    (fp_line (start -1.2 -1.2) (end -1.2 1.2)
+      (stroke (width 0.12) (type solid)) (layer "B.SilkS"))
+    (fp_line (start -1.2 1.2) (end 1.2 1.2)
+      (stroke (width 0.12) (type solid)) (layer "B.SilkS"))
+    (fp_line (start 1.2 -1.2) (end -1.2 -1.2)
+      (stroke (width 0.12) (type solid)) (layer "B.SilkS"))
+    (fp_line (start 1.2 1.2) (end 1.2 -1.2)
+      (stroke (width 0.12) (type solid)) (layer "B.SilkS"))
+    (fp_line (start -1.5 1.5) (end -1.5 -1.5)
+      (stroke (width 0.05) (type solid)) (layer "B.CrtYd"))
+    (fp_line (start -1.5 1.5) (end 1.5 1.5)
+      (stroke (width 0.05) (type solid)) (layer "B.CrtYd"))
+    (fp_line (start 1.5 -1.5) (end -1.5 -1.5)
+      (stroke (width 0.05) (type solid)) (layer "B.CrtYd"))
+    (fp_line (start 1.5 -1.5) (end 1.5 1.5)
+      (stroke (width 0.05) (type solid)) (layer "B.CrtYd"))
+    (pad "1" smd rect (at 0 0 180) (size 2 2) (layers "B.Cu" "B.Mask")
+      (net 10 "/CAN_L"))
+  )
   (footprint "Inductor_SMD:L_0402_1005Metric" (layer "B.Cu")
     (at 166.79 97.13 180)
@@
   (via (at 138 119) (size 0.8) (drill 0.4) (layers "F.Cu" "B.Cu") (free) (net 1))
   (via (at 138.8 90) (size 0.8) (drill 0.4) (layers "F.Cu" "B.Cu") (free) (net 1))
-  (via (at 166 119) (size 0.8) (drill 0.4) (layers "F.Cu" "B.Cu") (free) (net 1))
   (via (at 158.4 109.2) (size 0.45) (drill 0.2) (layers "F.Cu" "B.Cu") (free) (net 1))
   (via (at 169 109) (size 0.8) (drill 0.4) (layers "F.Cu" "B.Cu") (free) (net 1))
@@
   (segment (start 162.425 115.26) (end 162.425 117.0625) (width 0.2032) (layer "B.Cu") (net 10))
   (segment (start 162.095 115.26) (end 162.425 115.26) (width 0.2032) (layer "B.Cu") (net 10))
+  (segment (start 162.575 116.725) (end 160.9 118.4) (width 0.25) (layer "B.Cu") (net 10))
   (segment (start 163.2 112.82) (end 162.77 113.25) (width 0.2032) (layer "B.Cu") (net 10))
+  (segment (start 162.575 116.63) (end 162.575 116.725) (width 0.25) (layer "B.Cu") (net 10))
   (segment (start 161.6275 114.7925) (end 162.095 115.26) (width 0.2032) (layer "B.Cu") (net 10))
   (segment (start 163.2 111.9) (end 163.2 112.82) (width 0.2032) (layer "B.Cu") (net 10))
   (segment (start 161.6275 114.7925) (end 161.6275 113.6925) (width 0.2032) (layer "B.Cu") (net 10))
+  (segment (start 164.475 116.63) (end 164.475 116.775) (width 0.25) (layer "B.Cu") (net 11))
   (segment (start 163.85 112.815) (end 164.285 113.25) (width 0.2032) (layer "B.Cu") (net 11))
   (segment (start 163.85 111.9) (end 163.85 112.815) (width 0.2032) (layer "B.Cu") (net 11))
@@
   (segment (start 165.4275 113.6925) (end 165.4275 114.7925) (width 0.2032) (layer "B.Cu") (net 11))
   (segment (start 164.96 115.26) (end 164.625 115.26) (width 0.2032) (layer "B.Cu") (net 11))
+  (segment (start 164.475 116.775) (end 166.1 118.4) (width 0.25) (layer "B.Cu") (net 11))
   (segment (start 164.285 113.25) (end 164.985 113.25) (width 0.2032) (layer "B.Cu") (net 11))
   (segment (start 164.985 113.25) (end 165.4275 113.6925) (width 0.2032) (layer "B.Cu") (net 11))
